File: Ranger24/Ranger24.kicad_sch (KiCad schematic)
At the start: 36 parts, among them J1 LCD, J2 SPORT, J3 1051330011, J4 Flat Cable, Q1 MMBT3904, Q2 MMBT3904, Q3 PJA3441, U1 ESP32-WROOM-32D, U2 E28-2G4M27S, U4 CH340G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

Commit message: update
Parts:
- added C15: 0.1uF, Capacitor_SMD:C_0603_1608Metric, symbol Device:C_Small
- added U3: 78L05, Package_TO_SOT_SMD:SOT-23, symbol 78L05:78L05
Connections:
- net +5V: now also C15.2, U3.1 (OUT)
- net CPPM: now also J2.5 (Pin_5); no longer J2.1 (Pin_1)
- net GND: now also J2.2 (Pin_2), C15.1, U3.3 (GND); no longer J2.4 (Pin_4)
- net HB: now also J2.4 (Pin_4); no longer J2.2 (Pin_2)
- net S.PORT: now also J2.1 (Pin_1); no longer J2.5 (Pin_5)
- net VCC: now also U3.2 (IN)
Other:
- moved on the sheet: J2
