File: Ranger24/Ranger24.kicad_pcb (KiCad board)
At the start: 2 copper layers, 40.5 x 56 mm, 37 parts, among them J1 LCD, J2 SPORT, J3 1051330011, Q1 MMBT3904, Q2 MMBT3904, Q3 PJA3441, U1 ESP32-WROOM-32D, U2 E28-2G4M27S, U4 CH340G, U5 AMS1117-3.3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

Commit message: update
Parts:
- added C15: 0.1uF, Capacitor_SMD:C_0603_1608Metric, F.Cu at (155.0, 114.5)
- added U3: ~, Package_TO_SOT_SMD:SOT-23, F.Cu at (154.5, 112.1)
- J2: moved to B.Cu
- moved C7 1.82 mm to (146.6, 96.6), turned to 0 degrees
- moved R2 1.82 mm to (156.4, 96.6), turned to 180 degrees
Connections:
- J2 pad 1: /CPPM -> /S.PORT
- J2 pad 2: /HB -> GND
- J2 pad 4: GND -> /HB
- J2 pad 5: /S.PORT -> /CPPM
Routing:
- net +5V: track 2.50 -> 35.0 mm, vias 0 -> 2
- net /S.PORT: track 22.1 -> 36.1 mm, vias 1 -> 0
- net /VBAT: track 9.42 -> 15.7 mm, vias 0 -> 1
- net VCC: track 19.9 -> 23.8 mm
- net /LED: track 14.3 -> 15.2 mm
- net Net-(D4-DIN): track 2.40 -> 1.66 mm
- net GND: vias 168 -> 157

Commit message: update
edit screw holes
Routing:
- net /LED: track 15.2 -> 14.6 mm
- net GND: vias 157 -> 155
Other:
- outline, holes or cut-outs redrawn
Changed lines of the file:
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@@
 	(gr_circle
 		(center 168.941695 71.120091)
-		(end 170.74192 71.120091)
+		(end 169.941695 71.120091)
 		(stroke
 			(width 1)
@@
 	(gr_circle
 		(center 133.437258 122.126466)
-		(end 135.237483 122.126466)
+		(end 134.437258 122.126466)
 		(stroke
 			(width 1)
@@
 	(gr_circle
 		(center 133.437258 71.120091)
-		(end 135.237483 71.120091)
+		(end 134.437258 71.120091)
 		(stroke
 			(width 1)
@@
 	(gr_circle
 		(center 133.437258 71.120091)
-		(end 135.237483 71.120091)
+		(end 134.437258 71.120091)
 		(stroke
 			(width 1)
@@
 	(gr_circle
 		(center 168.941695 71.120091)
-		(end 170.74192 71.120091)
+		(end 169.941695 71.120091)
 		(stroke
 			(width 1)
@@
 	(gr_circle
 		(center 133.437258 122.126466)
-		(end 135.237483 122.126466)
+		(end 134.437258 122.126466)
 		(stroke
 			(width 1)
@@
 	(gr_circle
 		(center 168.946758 71.12328)
-		(end 170.746983 71.12328)
+		(end 169.946758 71.12328)
 		(stroke
 			(width 1)
@@
 	(gr_circle
 		(center 133.442321 122.129655)
-		(end 135.242546 122.129655)
+		(end 134.442321 122.129655)
 		(stroke
 			(width 1)
@@
 	(gr_circle
 		(center 133.442321 122.129655)
-		(end 135.242546 122.129655)
+		(end 134.442321 122.129655)
 		(stroke
 			(width 1)
@@
 	(gr_circle
 		(center 133.442321 71.12328)
-		(end 135.242546 71.12328)
+		(end 134.442321 71.12328)
 		(stroke
 			(width 1)
@@
 	(gr_circle
 		(center 133.442321 71.12328)
-		(end 135.242546 71.12328)
+		(end 134.442321 71.12328)
 		(stroke
 			(width 1)
@@
 	(gr_circle
 		(center 168.946758 71.12328)
-		(end 170.746983 71.12328)
+		(end 169.946758 71.12328)
 		(stroke
 			(width 1)
@@
 	(gr_circle
 		(center 133.46 122.13)
-		(end 135.26 122.13)
+		(end 134.46 122.13)
 		(locked yes)
 		(stroke
@@
 	(gr_circle
 		(center 133.46 71.13)
-		(end 135.26 71.13)
+		(end 134.46 71.13)
 		(locked yes)
 		(stroke
@@
 	(gr_circle
 		(center 168.96 71.13)
-		(end 170.76 71.13)
+		(end 169.96 71.13)
 		(locked yes)
 		(stroke
@@
 	)
 	(via
-		(at 158.1 99.1)
-		(size 0.6048)
-		(drill 0.3)
-		(layers "F.Cu" "B.Cu")
-		(free yes)
-		(net 2)
-	)
-	(via
 		(at 155.8 92.7)
 		(size 0.6048)
@@
 	)
 	(via
+		(at 160.6 100.2)
+		(size 0.6)
+		(drill 0.3)
+		(layers "F.Cu" "B.Cu")
+		(free yes)
+		(net 2)
+	)
+	(via
 		(at 145.2 75.2)
 		(size 0.6048)
@@
 	)
 	(via
-		(at 159.2 101.2)
-		(size 0.6048)
-		(drill 0.3)
-		(layers "F.Cu" "B.Cu")
-		(free yes)
-		(net 2)
-	)
-	(via
 		(at 148.33 117.97)
 		(size 0.6)
@@
 	)
 	(via
-		(at 160.6 102.4)
-		(size 0.6048)
-		(drill 0.3)
-		(layers "F.Cu" "B.Cu")
-		(free yes)
-		(net 2)
-	)
-	(via
 		(at 143.2 108.2)
 		(size 0.6048)
@@
 	)
 	(segment
-		(start 170.13 122.41)
-		(end 168.454 122.41)
-		(width 0.3048)
-		(layer "B.Cu")
-		(net 17)
-	)
-	(segment
-		(start 165.43 105.23)
-		(end 165.43 106.43)
+		(start 170.51 111.51)
+		(end 170.51 122.03)
 		(width 0.3048)
 		(layer "B.Cu")
@@
 	)
 	(segment
-		(start 155.94 95.74)
-		(end 165.43 105.23)
+		(start 155.94 94.14)
+		(end 155.94 96.94)
 		(width 0.3048)
 		(layer "B.Cu")
@@
 	)
 	(segment
-		(start 155.94 94.14)
-		(end 155.94 95.74)
+		(start 170.13 122.41)
+		(end 168.454 122.41)
 		(width 0.3048)
 		(layer "B.Cu")
@@
 	)
 	(segment
-		(start 170.51 111.51)
-		(end 170.51 122.03)
+		(start 155.94 96.94)
+		(end 170.51 111.51)
 		(width 0.3048)
 		(layer "B.Cu")
@@
 	)
 	(segment
-		(start 165.43 106.43)
-		(end 170.51 111.51)
-		(width 0.3048)
-		(layer "B.Cu")
-		(net 17)
-	)
-	(segment
 		(start 150.7682 87.87)
 		(end 156.33 87.87)
@@
 	)
 	(segment
-		(start 156.45 98.22)
-		(end 157.255 97.415)
+		(start 157.255 97.415)
+		(end 157.255 96.59)
 		(width 0.254)
 		(layer "F.Cu")
@@
 	)
 	(segment
-		(start 157.255 97.415)
-		(end 157.255 96.59)
+		(start 154.6 98.3)
+		(end 156.37 98.3)
 		(width 0.254)
 		(layer "F.Cu")
@@
 	)
 	(segment
-		(start 156.44 98.22)
-		(end 156.45 98.22)
+		(start 156.37 98.3)
+		(end 157.255 97.415)
 		(width 0.254)
 		(layer "F.Cu")
@@
 	)
 	(via
-		(at 156.44 98.22)
+		(at 154.6 98.3)
 		(size 0.6048)
 		(drill 0.3)
@@
 	)
 	(segment
-		(start 156.44 98.22)
-		(end 155.59 99.07)
+		(start 147.05 96.65)
+		(end 147.05 94.14)
 		(width 0.254)
 		(layer "B.Cu")
@@
 	)
 	(segment
-		(start 155.59 99.07)
-		(end 149.47 99.07)
+		(start 154.6 98.3)
+		(end 153.6 97.3)
 		(width 0.254)
 		(layer "B.Cu")
@@
 	)
 	(segment
-		(start 147.05 96.65)
-		(end 147.05 94.14)
+		(start 147.7 97.3)
+		(end 147.05 96.65)
 		(width 0.254)
 		(layer "B.Cu")
@@
 	)
 	(segment
-		(start 149.47 99.07)
-		(end 147.05 96.65)
+		(start 153.6 97.3)
+		(end 147.7 97.3)
 		(width 0.254)
 		(layer "B.Cu")
